File: breakouts/efm32wg/efm32wg.kicad_sch (KiCad schematic)
At the start: 1 part

Commit message: finish efm32wg board
Parts:
- added C1, C10, C11, C19, C2, C9: 10u, Capacitor_SMD:C_0805_2012Metric, symbol Device:C_Small
- added C12, C13, C14, C15, C16, C17, C5: 100n, Capacitor_SMD:C_0603_1608Metric, symbol Device:C_Small
- added C18, C8: 1u, Capacitor_SMD:C_0603_1608Metric, symbol Device:C_Small
- added C3, C4: 10p, Capacitor_SMD:C_0603_1608Metric, symbol Device:C_Small
- added C6, C7: 15p, Capacitor_SMD:C_0603_1608Metric, symbol Device:C_Small
- added D1: LED_RABG, Resistor_SMD:R_Array_Convex_2x0606, symbol Device:LED_RABG
- added F1, F2: 500mA, Fuse:Fuse_1206_3216Metric, symbol Device:Polyfuse_Small
- added J1: Target, extraparts:USB_Micro-B_U254-05, symbol Connector:USB_B_Micro
- added J2: DAPLink, extraparts:USB_Micro-B_U254-05, symbol Connector:USB_B_Micro
- added J3: PERIPH0, Connector_PinHeader_1.27mm:PinHeader_2x05_P1.27mm_Vertical_SMD, symbol Connector_Generic:Conn_02x05_Odd_Even
- added J4: PERIPH1, Connector_PinHeader_1.27mm:PinHeader_2x05_P1.27mm_Vertical_SMD, symbol Connector_Generic:Conn_02x05_Odd_Even
- added R1: DNP, Resistor_SMD:R_0603_1608Metric, symbol Device:R_Small
- added R10, R8, R9: 100, Resistor_SMD:R_0603_1608Metric, symbol Device:R_Small
- added R2, R3: 15, Resistor_SMD:R_0603_1608Metric, symbol Device:R_Small
- added R4, R5, R6, R7: 2k2, Resistor_SMD:R_0603_1608Metric, symbol Device:R_Small
- added SW1: BTN, Button_Switch_SMD:SW_SPST_PTS810, symbol Switch:SW_Push
- added U1: AZ1117CR2-3.3, Package_TO_SOT_SMD:SOT-89-3, symbol Regulator_Linear:AZ1117-3.3
- added Y1: 48MHz, Crystal:Crystal_SMD_TXC_7M-4Pin_3.2x2.5mm, symbol Device:Crystal_GND24_Small
- added Y2: 32.768kHz, Crystal:Crystal_SMD_MicroCrystal_CM9V-T1A-2Pin_1.6x1.0mm, symbol Device:Crystal_Small
- gave numbers to parts that had none: 1
Connections:
- net SDA0: now reaches U2.1 (PA0)
- net SDA0: now also J3.5 (Pin_5), R6.1
- net UART.RX: now reaches U2.11 (PC2)
- net UART.TX: now reaches U2.12 (PC3)
- net SDA1: now reaches U2.13 (PC4)
- net SDA1: now also J4.5 (Pin_5), R7.1
- net SCL1: now reaches U2.14 (PC5)
- net SCL1: now also J4.7 (Pin_7), R5.1
- net at U2.15 (PB7): now also C6.2, Y2.1
- net at U2.16 (PB8): now also C7.2, Y2.2
- net SCL0: now reaches U2.2 (PA1)
- net SCL0: now also J3.7 (Pin_7), R4.1
- net SWD.nRST: now reaches U2.20 (RESETn)
- net SWD.nRST: now also C5.2, R1.1
- net GND: now reaches U2.22 (VSS)
- net GND: now also U2.56 (VSS), U2.8 (VSS), C1.1, C10.2, C11.2, C12.2, C13.2, C14.2, C15.2, C16.2, C17.2, C18.2, C19.2, C2.2, C3.2, C4.1, C5.1, C6.1, C7.1, C8.1, C9.2, J1.5 (GND), J1.6 (Shield), J2.5 (GND), J2.6 (Shield), J3.3 (Pin_3), J4.3 (Pin_3), SW1.2, U1.1 (GND), Y1.2, Y1.4
- net +3V3: now reaches U2.23 (AVDD_1)
- net +3V3: now also U2.26 (IOVDD_3), U2.27 (AVDD_0), U2.39 (VDD_DREG), U2.55 (IOVDD_5), U2.7 (IOVDD_0), C10.1, C11.1, C12.1, C13.1, C14.1, C15.1, C16.1, C17.1, C2.1, C9.1, D1.2 (A), J3.1 (Pin_1), J4.1 (Pin_1), R1.2, R4.2, R5.2, R6.2, R7.2, U1.3 (VO)
- net at U2.24 (PB13): now also C3.1, Y1.1
- net at U2.25 (PB14): now also C4.2, Y1.3
- net MOSI1: now reaches U2.28 (PD0)
- net MOSI1: now also J4.2 (Pin_2)
- net MISO1: now reaches U2.29 (PD1)
- net MISO1: now also J4.4 (Pin_4)
- net SCK1: now reaches U2.30 (PD2)
- net SCK1: now also J4.6 (Pin_6)
- net CS1: now reaches U2.31 (PD3)
- net CS1: now also J4.8 (Pin_8)
- net TX1: now reaches U2.37 (PC6)
- net TX1: now also J4.9 (Pin_9)
- net RX1: now reaches U2.38 (PC7)
- net RX1: now also J4.10 (Pin_10)
- net at U2.40 (DECOUPLE): now also C8.2
- net LED_R: now reaches U2.41 (PC8)
- net LED_R: now also R8.1
- net LED_G: now reaches U2.42 (PC9)
- net LED_G: now also R9.1
- net LED_B: now reaches U2.43 (PC10)
- net LED_B: now also R10.1
- net BTN: now reaches U2.44 (PC11)
- net BTN: now also SW1.1
- net +5V: now reaches U2.45 (USB_VREGI)
- net +5V: now also U2.52 (USB_VBUS), C1.2, C19.1, F1.2, F2.2, U1.2 (VI)
- net at U2.46 (USB_VREGO): now also C18.1
- net at U2.47 (PF10): now also R2.1
- net at U2.48 (PF11): now also R3.1
- net SWD.SWCLK: now reaches U2.49 (PF0)
- net SWD.SWDIO: now reaches U2.50 (PF1)
- net SWD.SWO: now reaches U2.51 (PF2)
- net USB_ID: now reaches U2.53 (PF12)
- net USB_ID: now also J1.4 (ID)
- net MOSI0: now reaches U2.59 (PE10)
- net MOSI0: now also J3.2 (Pin_2)
- net MISO0: now reaches U2.60 (PE11)
- net MISO0: now also J3.4 (Pin_4)
- net SCK0: now reaches U2.61 (PE12)
- net SCK0: now also J3.6 (Pin_6)
- net CS0: now reaches U2.62 (PE13)
- net CS0: now also J3.8 (Pin_8)
- net TX0: now reaches U2.63 (PE14)
- net TX0: now also J3.9 (Pin_9)
- net RX0: now reaches U2.64 (PE15)
- net RX0: now also J3.10 (Pin_10)
- new net: D1.1 (RK), R8.2
- new net: D1.3 (BK), R10.2
- new net: D1.4 (GK), R9.2
- new net: F2.1, J2.1 (VBUS)
- new net: F1.1, J1.1 (VBUS)
- new net DAP.D+: J2.3 (D+)
- new net DAP.D-: J2.2 (D-)
- new net USB_D+: J1.3 (D+), R3.2
- new net USB_D-: J1.2 (D-), R2.2
- no-connect marks 0 -> 20
Other:
- sheet DAPLink ports: added JTAG{JTAG}, SWD{SWD}, UART{UART}, USB{USB}; removed none
- note added: "AVDD"
- note added: "I2C0"
- note added: "I2C1"
- note added: "IOVDD"
- note added: "LEUART0"
- note added: "LEUART1"
- note added: "Note CR2 package!"
- note added: "RX"
- note added: "TIM2"
- note added: "TX"
- note added: "USART0"
- note added: "USART1"
- note added: "USART2"
- note added: "VDD_DREG"
