File: breakouts/ft4232h/ft4232h.kicad_sch (KiCad schematic)
At the start: 67 parts, among them J1 USB, J2 standard0, J3 standard1, U1 LD39020ATPU33R, U2 93LCxxBxxOT, U3 FT4232H, U4 LD39020ATPU33R, U5 LD39020ATPU33R, Y1 12MHz

Commit message: move to KiCad 7
Other:
- note added: "For JTAG, populate R18, R19, R20, R21, R22. To switch to SWD, depopulate R18, R20, and R21 and populate R16 and R17."
- note added: "For JTAG, populate R25, R26, R27, R28, R29. To switch to SWD, depopulate R25, R27, and R28 and populate R23 and R24."
- note removed: "For JTAG, populate R18, R19, R20, R21, R22. To switch to SWD, depopulate R20 and R21 and populate R16 and R17."
- note removed: "For JTAG, populate R25, R26, R27, R28, R29. To switch to SWD, depopulate R27 and R28 and populate R23 and R24."

Commit message: small updates from bringup from months ago
Parts:
- R16, R17, R25, R27, R28: now not fitted
Changed lines of the file:
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@@
   )
   (symbol (lib_id "Device:R_Small") (at 267.335 124.46 90) (unit 1)
-    (in_bom yes) (on_board yes) (dnp no)
+    (in_bom yes) (on_board yes) (dnp yes)
     (property "Reference" "R28" (at 271.145 123.19 90)
       (effects (font (size 1.27 1.27)))
@@
   )
   (symbol (lib_id "Device:R_Small") (at 267.335 116.84 90) (unit 1)
-    (in_bom yes) (on_board yes) (dnp no)
+    (in_bom yes) (on_board yes) (dnp yes)
     (property "Reference" "R25" (at 271.145 115.57 90)
       (effects (font (size 1.27 1.27)))
@@
   )
   (symbol (lib_id "Device:R_Small") (at 267.335 78.105 90) (unit 1)
-    (in_bom yes) (on_board yes) (dnp no)
+    (in_bom yes) (on_board yes) (dnp yes)
     (property "Reference" "R16" (at 271.145 76.835 90)
       (effects (font (size 1.27 1.27)))
@@
   )
   (symbol (lib_id "Device:R_Small") (at 267.335 121.92 90) (unit 1)
-    (in_bom yes) (on_board yes) (dnp no)
+    (in_bom yes) (on_board yes) (dnp yes)
     (property "Reference" "R27" (at 271.145 120.65 90)
       (effects (font (size 1.27 1.27)))
@@
   )
   (symbol (lib_id "Device:R_Small") (at 267.335 80.645 90) (unit 1)
-    (in_bom yes) (on_board yes) (dnp no)
+    (in_bom yes) (on_board yes) (dnp yes)
     (property "Reference" "R17" (at 271.145 79.375 90)
       (effects (font (size 1.27 1.27)))
