File: breakouts/usb_pdmon/usb_pdmon.kicad_pcb (KiCad board)
At the start: 2 copper layers, 32 x 32 mm, 42 parts, among them J1 SWD/UART, J2 USB_C_Receptacle_USB2.0, J3 LIN, Q1 DMP3099L, Q2 DMP3099L, Q3 MMBT2222, Q4 DMP3099L, Q5 DMP3099L, Q6 MMBT2222, Q7 MMBT2222, SW1 boot, U1 AP7381-33Y, U2 CH32X035GxUx, U3 ACS70331

Commit message: add usb_c_splitter
Other:
- board text added: "1 nc 2 nc 3 gnd 4 lin 5 gnd"
- board text added: "nc 6 nc 7 vbus 8 vbus 9"
- board text added: "usb_pdmon matt tran"
Changed lines of the file:
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@@
     )
   )
+  (gr_line (start 157.5 96.5) (end 158.75 97.75)
+    (stroke (width 0.15) (type solid)) (layer "B.SilkS"))
+  (gr_line (start 156.5 103.5) (end 157.5 103.5)
+    (stroke (width 0.15) (type solid)) (layer "B.SilkS"))
+  (gr_line (start 158.75 102.25) (end 158.75 97.75)
+    (stroke (width 0.15) (type solid)) (layer "B.SilkS"))
+  (gr_line (start 156.5 96.5) (end 157.5 96.5)
+    (stroke (width 0.15) (type solid)) (layer "B.SilkS"))
+  (gr_line (start 156.5 96.5) (end 156.5 103.5)
+    (stroke (width 0.15) (type solid)) (layer "B.SilkS"))
+  (gr_line (start 157.5 103.5) (end 158.75 102.25)
+    (stroke (width 0.15) (type solid)) (layer "B.SilkS"))
   (gr_arc (start 172.75 84) (mid 173.103553 84.146447) (end 173.25 84.5)
     (stroke (width 0.1) (type default)) (layer "Edge.Cuts"))
@@
   (gr_arc (start 173.25 115.5) (mid 173.103553 115.853553) (end 172.75 116)
     (stroke (width 0.1) (type default)) (layer "Edge.Cuts"))
+  (gr_text "1 nc\n2 nc\n3 gnd\n4 lin\n5 gnd" (at 157.5 100) (layer "B.SilkS")
+    (effects (font (size 0.8 0.8) (thickness 0.15)) (justify left mirror))
+  )
+  (gr_text "usb_pdmon\nmatt tran" (at 142.25 115) (layer "B.SilkS")
+    (effects (font (size 0.8 0.8) (thickness 0.15)) (justify right bottom mirror))
+  )
+  (gr_text "nc 6\nnc 7\nvbus 8\nvbus 9" (at 157.75 100) (layer "B.SilkS")
+    (effects (font (size 0.8 0.8) (thickness 0.15)) (justify right mirror))
+  )
   (segment (start 149.175 114.5) (end 149.175 113.05) (width 0.3048) (layer "F.Cu") (net 1))
   (segment (start 149.175 113.05) (end 149.225 113) (width 0.3048) (layer "F.Cu") (net 1))
@@
         (xy 148.75 97.25)
         (xy 148.75 102.75)
-        (xy 148.75 102.75)
         (xy 150.5 104.5)

Commit message: update usb_pdmon schematic values
Parts:
- R12: value 150k -> 12k
- R13: value 100k -> 10k
Changed lines of the file:
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@@
         (effects (font (size 0.4 0.4) (thickness 0.1)))
     )
-    (fp_text value "150k" (at 0 1.17) (layer "F.Fab")
+    (fp_text value "12k" (at 0 1.17) (layer "F.Fab")
         (effects (font (size 1 1) (thickness 0.15)))
     )
@@
         (effects (font (size 0.4 0.4) (thickness 0.1)))
     )
-    (fp_text value "100k" (at 0 1.43) (layer "F.Fab")
-        (effects (font (size 1 1) (thickness 0.15)))
-    )
+    (fp_text value "10k" (at 0 1.43) (layer "F.Fab")
+        (effects (font (size 1 1) (thickness 0.15)))
+    )
