File: projects/keyboard/keyboard.kicad_sch (KiCad schematic)
At the start: 47 parts, among them J1 USB_C, J2 SWD, J3 lipo, J4 ICSP, Q1 PSMN4R5-30YLC, SW1 spinny boi, SW2 pwr, U1 RPi_Pico, U3 SSD1306, U4 ATtiny13A-SS, U5 MIC5019, U6 MCP73831-2-OT

Commit message: finished keyboard layout
Parts:
- removed FB1: FerriteBead_Small, Capacitor_SMD:C_0402_1005Metric, symbol Device:FerriteBead_Small
- removed SW2: pwr, Button_Switch_Keyboard:SW_Cherry_MX_1.00u_PCB, symbol Switch:SW_SPST
Connections:
- net GND: now also J1.S1 (SHIELD), R16.2, SW1.S1; no longer D5.1 (K), SW1.S2
- net enc_a: now also SW1.B; no longer SW1.A
- net enc_b: now also SW1.A; no longer SW1.B
- net led_r0: now also U1.2 (GP1); no longer U1.1 (GP0)
- net led_r1: now also U1.5 (GP3); no longer U1.4 (GP2)
- net led_r2: now also U1.7 (GP5); no longer U1.6 (GP4)
- net led_r3: now also U1.10 (GP7); no longer U1.9 (GP6)
- net led_r4: now also U1.12 (GP9); no longer U1.11 (GP8)
- net lipo+: now also R15.1; no longer D4.2 (A)
- net pwr_en: now also U4.3 (PB4); no longer J4.2 (Pin_2), U4.5 (PB0)
- net pwr_led: now also D4.1 (K), D5.2 (A), J4.2 (Pin_2), U4.5 (PB0); no longer R15.2, R16.1, U4.3 (PB4)
- net pwr_sw: now also SW1.S2
- net sw_r0: now also U1.1 (GP0); no longer U1.2 (GP1)
- net sw_r1: now also U1.4 (GP2); no longer U1.5 (GP3)
- net sw_r2: now also U1.6 (GP4); no longer U1.7 (GP5)
- net sw_r3: now also U1.9 (GP6); no longer U1.10 (GP7)
- net sw_r4: now also U1.11 (GP8); no longer U1.12 (GP9)
- net vbatt_sense: now also U4.2 (PB3); no longer J4.4 (Pin_4), U4.7 (PB2)
- net watchdog: now also J4.4 (Pin_4), U4.7 (PB2); no longer U4.2 (PB3)
- net enc_sw: no longer names the net of U1.29 (GP22)
- net enc_sw: no longer SW1.S1
- new net: D5.1 (K), R16.1
- new net: D4.2 (A), R15.2
- no-connect marks 16 -> 17
Other:
- moved on the sheet: D4, D5, R15, R16, SW1

Commit message: small updates from bringup from months ago
Parts:
- D5, R16: now not fitted
Changed lines of the file:
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@@
   )
   (symbol (lib_id "Device:LED_Small") (at 259.08 46.355 180) (unit 1)
-    (in_bom yes) (on_board yes) (dnp no)
+    (in_bom yes) (on_board yes) (dnp yes)
     (property "Reference" "D5" (at 257.81 42.545 0)
       (effects (font (size 1.27 1.27)) (justify right))
@@
   )
   (symbol (lib_id "Device:R_Small") (at 265.43 46.355 90) (unit 1)
-    (in_bom yes) (on_board yes) (dnp no)
+    (in_bom yes) (on_board yes) (dnp yes)
     (property "Reference" "R16" (at 267.335 42.545 90)
       (effects (font (size 1.27 1.27)) (justify left))
