File: projects/lightsaber/blade/blade.kicad_pcb (KiCad board)
At the start: 2 copper layers, 22.2 x 22.2 mm, 1 part, among them J1 blade

Commit message: move to KiCad 7
Changed lines of the file:
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@@
-(kicad_pcb (version 20211014) (generator pcbnew)
+(kicad_pcb (version 20221018) (generator pcbnew)
   (general
     (thickness 1.6)
@@
     (pcbplotparams
       (layerselection 0x00010fc_ffffffff)
+      (plot_on_all_layers_selection 0x0000000_00000000)
       (disableapertmacros false)
       (usegerberextensions false)
@@
       (usegerberadvancedattributes true)
       (creategerberjobfile true)
-      (svguseinch false)
+      (dashed_line_dash_ratio 12.000000)
+      (dashed_line_gap_ratio 3.000000)
       (svgprecision 6)
-      (excludeedgelayer true)
       (plotframeref false)
       (viasonmask false)
@@
     (attr smd exclude_from_pos_files)
     (fp_text reference "J1" (at 0 -10.45) (layer "B.SilkS")
-      (effects (font (size 0.4 0.4) (thickness 0.1)) (justify mirror))
+        (effects (font (size 0.4 0.4) (thickness 0.1)) (justify mirror))
     )
     (fp_text value "blade" (at 0 11.75) (layer "F.Fab")
-      (effects (font (size 1 1) (thickness 0.15)))
+        (effects (font (size 1 1) (thickness 0.15)))
     )
-    (fp_circle (center 0 0) (end 9.5 0) (layer "B.SilkS") (width 0.1) (fill none))
-    (fp_circle (center 0 0) (end 2.8 0) (layer "B.SilkS") (width 0.1) (fill none))
-    (fp_circle (center 0 0) (end 2.8 0) (layer "F.SilkS") (width 0.1) (fill none))
-    (pad "" np_thru_hole circle (at 0 0) (size 2.8 2.8) (drill 2.8) (layers F&B.Cu *.Mask)
+    (fp_circle (center 0 0) (end 2.8 0)
+      (stroke (width 0.1) (type solid)) (fill none) (layer "B.SilkS"))
+    (fp_circle (center 0 0) (end 9.5 0)
+      (stroke (width 0.1) (type solid)) (fill none) (layer "B.SilkS"))
+    (fp_circle (center 0 0) (end 2.8 0)
+      (stroke (width 0.1) (type solid)) (fill none) (layer "F.SilkS"))
+    (pad "" np_thru_hole circle (at 0 0) (size 2.8 2.8) (drill 2.8) (layers "F&B.Cu" "*.Mask")
       (net 1 "/gnd"))
-    (pad "1" smd custom (at 0 0) (size 0 0) (layers "F.Cu" "F.Mask")
-      (net 1 "/gnd") (pinfunction "Pin_1") (pintype "passive")
+    (pad "1" smd custom (at 0 0) (size 0.001 0.001) (layers "F.Cu" "F.Mask")
+      (net 1 "/gnd") (pinfunction "Pin_1") (pintype "passive") (thermal_bridge_angle 45)
       (options (clearance outline) (anchor circle))
       (primitives
-        (gr_circle (center 0 0) (end 4 0) (width 2))
+        (gr_circle (center 0 0) (end 4 0) (width 2) (fill none))
       ))
     (pad "1" smd custom (at 0 7.75) (size 1.524 1.524) (layers "B.Cu" "B.Mask")
-      (net 1 "/gnd") (pinfunction "Pin_1") (pintype "passive")
+      (net 1 "/gnd") (pinfunction "Pin_1") (pintype "passive") (thermal_bridge_angle 45)
       (options (clearance outline) (anchor circle))
       (primitives
-        (gr_poly (pts
+        (gr_poly
+          (pts
             (arc (start -5.306355 -15.327055) (mid -0.000108 1.500612) (end 5.305222 -15.327344))
             (arc (start 3.584493 -12.869888) (mid -0.000963 -1.499388) (end -3.584225 -12.870579))
-          ) (width 0.01) (fill yes))
+          )
+          (width 0.01) (fill yes))
       ))
-    (pad "2" smd custom (at 0 0) (size 0 0) (layers "F.Cu" "F.Mask")
-      (net 1 "/gnd") (pinfunction "Pin_2") (pintype "passive")
+    (pad "2" smd custom (at 0 0) (size 0.001 0.001) (layers "F.Cu" "F.Mask")
+      (net 1 "/gnd") (pinfunction "Pin_2") (pintype "passive") (thermal_bridge_angle 45)
       (options (clearance outline) (anchor circle))
       (primitives
-        (gr_circle (center 0 0) (end 6.55 0) (width 2.6))
+        (gr_circle (center 0 0) (end 6.55 0) (width 2.6) (fill none))
       ))
     (pad "2" smd custom (at 0 4.5) (size 1.524 1.524) (layers "B.Cu" "B.Mask")
-      (net 1 "/gnd") (pinfunction "Pin_2") (pintype "passive")
+      (net 1 "/gnd") (pinfunction "Pin_2") (pintype "passive") (thermal_bridge_angle 45)
       (options (clearance outline) (anchor circle))
       (primitives
-        (gr_poly (pts
+        (gr_poly
+          (pts
             (arc (start -1.720641 -6.957518) (mid -0.000054 -1.5) (end 1.720729 -6.957456))
             (arc (start 3.441099 -9.4151) (mid 0.000199 1.500612) (end -3.442734 -9.414458))
-          ) (width 0.01) (fill yes))
+          )
+          (width 0.01) (fill yes))
       ))
-    (pad "3" smd custom (at 0 0) (size 0 0) (layers "F.Cu" "F.Mask")
-      (net 1 "/gnd") (pinfunction "Pin_3") (pintype "passive")
+    (pad "3" smd custom (at 0 -4) (size 1.524 1.524) (layers "B.Cu" "B.Mask")
+      (net 1 "/gnd") (pinfunction "Pin_3") (pintype "passive") (thermal_bridge_angle 45)
       (options (clearance outline) (anchor circle))
       (primitives
-        (gr_circle (center 0 0) (end 9.4 0) (width 2.6))
+        (gr_poly
+          (pts
+            (arc (start 1.268065 1.281175) (mid 0.000116 1) (end -1.267855 1.281077))
+            (arc (start -3.909219 -4.383347) (mid -0.001678 -5.25) (end 3.906178 -4.384765))
+          )
+          (width 0.01) (fill yes))
       ))
-    (pad "3" smd custom (at 0 -4) (size 1.524 1.524) (layers "B.Cu" "B.Mask")
-      (net 1 "/gnd") (pinfunction "Pin_3") (pintype "passive")
+    (pad "3" smd custom (at 0 0) (size 0.001 0.001) (layers "F.Cu" "F.Mask")
+      (net 1 "/gnd") (pinfunction "Pin_3") (pintype "passive") (thermal_bridge_angle 45)
       (options (clearance outline) (anchor circle))
       (primitives
-        (gr_poly (pts
-            (arc (start 1.268065 1.281175) (mid 0.000116 1) (end -1.267855 1.281077))
-            (arc (start -3.909219 -4.383347) (mid -0.001678 -5.25) (end 3.906178 -4.384765))
-          ) (width 0.01) (fill yes))
+        (gr_circle (center 0 0) (end 9.4 0) (width 2.6) (fill none))
       ))
   )
-  (gr_circle (center 147.75 98.25) (end 158.85 98.25) (layer "Edge.Cuts") (width 0.1) (fill none))
+  (gr_circle (center 147.75 98.25) (end 158.85 98.25)
+    (stroke (width 0.1) (type solid)) (fill none) (layer "Edge.Cuts"))
   (gr_text "vbatt" (at 147.75 100.55) (layer "B.SilkS")
     (effects (font (size 0.4 0.4) (thickness 0.1)) (justify mirror))

Commit message: update kicad 8.0.0
Connections:
- J1 pad : /gnd -> (no net)
