File: projects/rvice_adc/fpga.kicad_sch (KiCad schematic)
At the start: 28 parts, among them U6 W25Q32JVSS

Commit message: wip rvice_adc layout
Parts:
- added C?: 100n, Capacitor_SMD:C_0402_1005Metric, symbol Device:C_Small
Connections:
- net +1V2: now also C?.1
- net GND: now also C?.2
- net led_b: now also U?.40 (RGB1); no longer U?.41 (RGB2)
- net led_g: now also U?.41 (RGB2); no longer U?.40 (RGB1)
- net sdo1: now also U?.36 (IOT_48b); no longer U?.23 (IOT_37a)
- net sdo2: now also U?.34 (IOT_44b); no longer U?.25 (IOT_36b)
- net sdo3: now also U?.32 (IOT_43a); no longer U?.26 (IOT_39a)
- net sdo4: now also U?.31 (IOT_42b); no longer U?.27 (IOT_38b)
- net sdo6: now also U?.27 (IOT_38b); no longer U?.31 (IOT_42b)
- net sdo7: now also U?.26 (IOT_39a); no longer U?.32 (IOT_43a)
- net sdo8: now also U?.25 (IOT_36b); no longer U?.34 (IOT_44b)
- net spi2.cs: now also U?.48 (IOB_4a); no longer U?.18 (IOB_31b)
- net spi2.miso: now also U?.46 (IOB_0a); no longer U?.20 (IOB_25b_G3)
- net spi2.mosi: now also U?.45 (IOB_5b); no longer U?.21 (IOB_23b)
- net spi2.sck: now also U?.47 (IOB_2a); no longer U?.19 (IOB_29b)
- net ~{cnv}: now also U?.38 (IOT_50b); no longer U?.36 (IOT_48b)

Commit message: update kicad 8.0.0
Parts:
- gave numbers to parts that had none: 25
