File: projects/rvice_adc/rvice_adc.kicad_pcb (KiCad board)
At the start: 2 copper layers, 119 parts, among them J1 USB1, J10 ain8, J11 SWD/UART, J2 USB2, J3 ain1, J4 ain2, J5 ain3, J6 ain4, J7 ain5, J8 ain6, J9 ain7, SW1 btn1, SW2 btn1, U1 AP3401, U2 AP3401, U3 AP3401, U4 CH32V203CxTx, U5 ICE5LP1K-SG48, U6 W25Q32JVSS, U7 LTC2320-16, Y1 8MHz

Commit message: wip rvice_adc layout
Parts:
- added C48: 100n, Capacitor_SMD:C_0402_1005Metric, B.Cu at (156.5, 111.8)
- added C49: 100n, Capacitor_SMD:C_0402_1005Metric, B.Cu at (158.2, 114.2)
- added C50: 100n, Capacitor_SMD:C_0402_1005Metric, B.Cu at (161.2, 105.8)
- added C51: 100n, Capacitor_SMD:C_0402_1005Metric, B.Cu at (163.2, 105.8)
- added C52: 100n, Capacitor_SMD:C_0402_1005Metric, B.Cu at (146.2, 109.2)
- C10, C11, C12, C13, C14, C15, C16, C17, C2, C20, C21, C22, C23, C24, C25, C26, C27, C28, C30, C31, C32, C33, C34, C35, C36, C37, C38, C39, C4, C40, C41, C43, C44, C45, C46, C47, C6, C8, C9, F1, J10, J4, J6, J8, R11, R12, R15, R16, R17, R18, R19, R20, R21, R22, R23, R24, R25, R26, R27, R3, R31, R32, R33, R34, R35, R4, R42, R43, R7, R8, U1, U2, U3: moved to B.Cu
- L1, L2, L3: footprint Inductor_SMD:L_Taiyo-Yuden_NR-30xx -> Inductor_SMD:L_Walsin_WLFM201609x; moved to B.Cu
- moved C12 117.9 mm to (135.0, 118.8)
- moved R20 113.8 mm to (135.0, 119.8)
- moved R21 113.7 mm to (135.0, 120.8), turned to 180 degrees
- moved C35 113.1 mm to (146.2, 106.2)
- moved C36 112.8 mm to (146.2, 107.2), turned to 180 degrees
- moved U1 111.3 mm to (137.8, 120.2), turned to -90 degrees
- moved R17 111.1 mm to (135.0, 121.8)
- moved C29 111.0 mm to (144.8, 118.5), turned to -90 degrees
- moved C13 110.4 mm to (142.2, 118.8)
- moved C32 110.3 mm to (146.2, 108.2)
- moved R23 109.6 mm to (142.2, 120.8), turned to 180 degrees
- moved C33 107.1 mm to (150.8, 113.8), turned to 90 degrees
- moved R22 106.3 mm to (142.2, 119.8)
- moved L1 105.8 mm to (137.8, 116.8), turned to 180 degrees
- moved C34 105.6 mm to (151.8, 113.8), turned to -90 degrees
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Connections:
- C1 pad 1: /a1.in+ -> /a1.in-
- C1 pad 2: /a1.in- -> /a1.in+
- C3 pad 1: /a3.in+ -> /a3.in-
- C3 pad 2: /a3.in- -> /a3.in+
- C5 pad 1: /a5.in+ -> /a5.in-
- C5 pad 2: /a5.in- -> /a5.in+
- C7 pad 1: /a7.in+ -> /a7.in-
- C7 pad 2: /a7.in- -> /a7.in+
- J11 pad 10: /micro/swdio -> /micro/~{rst}
- J11 pad 2: GND -> /micro/swdio
- J11 pad 3: /micro/rx -> GND
- J11 pad 4: /micro/tx -> /micro/swclk
- J11 pad 5: GND -> /micro/rx
- J11 pad 6: /micro/~{rst} -> unconnected-(J11-Pin_6-Pad6)
- J11 pad 7: unconnected-(J11-Pin_7-Pad7) -> /micro/tx
- J11 pad 9: /micro/swclk -> GND
- R1 pad 1: /a1.in+ -> /a1.in-
- R10 pad 1: /a5.in- -> /a5.in+
- R13 pad 1: /a7.in+ -> /a7.in-
- R14 pad 1: /a7.in- -> /a7.in+
- R2 pad 1: /a1.in- -> /a1.in+
- R35 pad 2: /micro/cdone -> /fpga/cdone
- R5 pad 1: /a3.in+ -> /a3.in-
- R6 pad 1: /a3.in- -> /a3.in+
- R9 pad 1: /a5.in+ -> /a5.in-
- U4 pad 10: /micro/btn1 -> /fpga/flash.sck
- U4 pad 11: unconnected-(U4-PA1/ADC1-Pad11) -> /fpga/flash.mosi
- U4 pad 12: unconnected-(U4-PA2/ADC2-Pad12) -> /fpga/flash.cs
- U4 pad 13: unconnected-(U4-PA3/ADC3-Pad13) -> /fpga/flash.miso
- U4 pad 14: /fpga/creset -> /fpga/spi1.cs
- U4 pad 15: /micro/cdone -> /fpga/spi1.sck
- U4 pad 16: /fpga/flash.mosi -> /fpga/spi1.miso
- U4 pad 17: /fpga/flash.miso -> /fpga/spi1.mosi
- U4 pad 18: /fpga/flash.sck -> /fpga/creset
- U4 pad 19: /fpga/flash.cs -> /fpga/cdone
- U4 pad 3: /micro/led_g -> /micro/led_b
- U4 pad 38: /fpga/spi1.cs -> unconnected-(U4-PA15-Pad38)
- U4 pad 39: /fpga/spi1.sck -> unconnected-(U4-PB3-Pad39)
- U4 pad 4: /micro/led_b -> /micro/led_g
- U4 pad 40: /fpga/spi1.miso -> unconnected-(U4-PB4-Pad40)
- U4 pad 41: /fpga/spi1.mosi -> unconnected-(U4-PB5-Pad41)
- U4 pad 46: unconnected-(U4-PB9-Pad46) -> /micro/btn1
- U5 pad 18: /fpga/spi2.cs -> unconnected-(U5B-IOB_31b-Pad18)
- U5 pad 19: /fpga/spi2.sck -> unconnected-(U5B-IOB_29b-Pad19)
- U5 pad 20: /fpga/spi2.miso -> unconnected-(U5B-IOB_25b_G3-Pad20)
- U5 pad 21: /fpga/spi2.mosi -> unconnected-(U5B-IOB_23b-Pad21)
- U5 pad 23: /adc/sdo1 -> unconnected-(U5A-IOT_37a-Pad23)
- U5 pad 25: /adc/sdo2 -> /adc/sdo8
- U5 pad 26: /adc/sdo3 -> /adc/sdo7
- U5 pad 27: /adc/sdo4 -> /adc/sdo6
- U5 pad 31: /adc/sdo6 -> /adc/sdo4
- U5 pad 32: /adc/sdo7 -> /adc/sdo3
- U5 pad 34: /adc/sdo8 -> /adc/sdo2
- U5 pad 36: /adc/~{cnv} -> /adc/sdo1
- U5 pad 38: unconnected-(U5A-IOT_50b-Pad38) -> /adc/~{cnv}
- U5 pad 40: /fpga/led_g -> /fpga/led_b
- U5 pad 41: /fpga/led_b -> /fpga/led_g
- U5 pad 45: unconnected-(U5C-IOB_5b-Pad45) -> /fpga/spi2.mosi
- U5 pad 46: unconnected-(U5C-IOB_0a-Pad46) -> /fpga/spi2.miso
- U5 pad 47: unconnected-(U5C-IOB_2a-Pad47) -> /fpga/spi2.sck
- U5 pad 48: unconnected-(U5C-IOB_4a-Pad48) -> /fpga/spi2.cs
- U5 pad 7: /micro/cdone -> /fpga/cdone
Routing:
- net +3V3: track 0.00 -> 85.0 mm, vias 0 -> 10
- net +5V: track 0.00 -> 46.0 mm, vias 0 -> 3
- net +2V5: track 0.00 -> 39.4 mm, vias 0 -> 6
- net +1V2: track 0.00 -> 34.2 mm, vias 0 -> 2
- net /adc/vdd: track 0.00 -> 31.2 mm, vias 0 -> 5
- net /vbus: track 0.00 -> 21.2 mm, vias 0 -> 2
- net /micro/~{rst}: track 0.00 -> 20.0 mm, vias 0 -> 2
- net /adc/clkin: track 0.00 -> 15.2 mm, vias 0 -> 2
- net /fpga/flash.cs: track 0.00 -> 14.7 mm, vias 0 -> 2
- net /fpga/flash.miso: track 0.00 -> 13.7 mm, vias 0 -> 2
- net /micro/swclk: track 0.00 -> 13.0 mm, vias 0 -> 2
- net /fpga/clk: track 0.00 -> 11.6 mm
- net /fpga/flash.sck: track 0.00 -> 10.9 mm
- net /power/pg_3v3: track 0.00 -> 10.7 mm, vias 0 -> 2
- net /power/pg_1v2: track 0.00 -> 10.7 mm, vias 0 -> 2
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- added copper zone on B.Cu, net GND
- added copper zone on F.Cu, net GND
Other:
- board outline added: 44 x 27 mm

Commit message: rvice_adc layout done
Routing:
- net GND: vias 0 -> 319
Other:
- board text added: "+"
- board text added: "-"
- board text added: "0.2mm edge clearance instead of required 15mil (0.381mm), to test"
- board text added: "ain1"
- board text added: "ain2"
- board text added: "ain3"
- board text added: "ain4"
- board text added: "ain5"
- board text added: "ain6"
- board text added: "ain7"
- board text added: "ain8"
- board text added: "rvice_adc - matt tran"
