File: projects/rvice_adc/rvice_adc.kicad_sch (KiCad schematic)
At the start: 35 parts, among them J1 USB1, J10 ain8, J2 USB2, J3 ain1, J4 ain2, J5 ain3, J6 ain4, J7 ain5, J8 ain6, J9 ain7

Commit message: wip rvice_adc layout
Connections:
- net a1.in+: now also C1.2, R2.1; no longer C1.1, R1.1
- net a1.in-: now also C1.1, R1.1; no longer C1.2, R2.1
- net a3.in+: now also C3.2, R6.1; no longer C3.1, R5.1
- net a3.in-: now also C3.1, R5.1; no longer C3.2, R6.1
- net a5.in+: now also C5.2, R10.1; no longer C5.1, R9.1
- net a5.in-: now also C5.1, R9.1; no longer C5.2, R10.1
- net a7.in+: now also C7.2, R14.1; no longer C7.1, R13.1
- net a7.in-: now also C7.1, R13.1; no longer C7.2, R14.1
Changed lines of the file:
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@@
     (effects (font (size 1.27 1.27)) (justify right bottom))
   )
-  (label "a1.in+" (at 196.85 69.85 180) (fields_autoplaced)
+  (label "a1.in+" (at 196.85 74.93 180) (fields_autoplaced)
     (effects (font (size 1.27 1.27)) (justify right bottom))
   )
@@
     (effects (font (size 1.27 1.27)) (justify right bottom))
   )
-  (label "a7.in+" (at 241.3 105.41 180) (fields_autoplaced)
+  (label "a7.in+" (at 241.3 110.49 180) (fields_autoplaced)
     (effects (font (size 1.27 1.27)) (justify right bottom))
   )
@@
     (effects (font (size 1.27 1.27)) (justify right bottom))
   )
-  (label "a5.in-" (at 241.3 74.93 180) (fields_autoplaced)
+  (label "a5.in-" (at 241.3 69.85 180) (fields_autoplaced)
     (effects (font (size 1.27 1.27)) (justify right bottom))
   )
@@
     (effects (font (size 1.27 1.27)) (justify left bottom))
   )
-  (label "a1.in-" (at 196.85 74.93 180) (fields_autoplaced)
+  (label "a1.in-" (at 196.85 69.85 180) (fields_autoplaced)
     (effects (font (size 1.27 1.27)) (justify right bottom))
   )
@@
     (effects (font (size 1.27 1.27)) (justify right bottom))
   )
-  (label "usb1.d+" (at 44.45 87.63 0)
+  (label "usb1.d+" (at 44.45 87.63 0) (fields_autoplaced)
     (effects (font (size 1.27 1.27)) (justify left bottom))
   )
-  (label "a5.in+" (at 241.3 69.85 180) (fields_autoplaced)
+  (label "a5.in+" (at 241.3 74.93 180) (fields_autoplaced)
     (effects (font (size 1.27 1.27)) (justify right bottom))
   )
@@
     (effects (font (size 1.27 1.27)) (justify right bottom))
   )
-  (label "a7.in-" (at 241.3 110.49 180) (fields_autoplaced)
+  (label "a7.in-" (at 241.3 105.41 180) (fields_autoplaced)
     (effects (font (size 1.27 1.27)) (justify right bottom))
   )
-  (label "a3.in+" (at 196.85 105.41 180) (fields_autoplaced)
+  (label "a3.in+" (at 196.85 110.49 180) (fields_autoplaced)
     (effects (font (size 1.27 1.27)) (justify right bottom))
   )
@@
     (effects (font (size 1.27 1.27)) (justify right bottom))
   )
-  (label "a3.in-" (at 196.85 110.49 180) (fields_autoplaced)
+  (label "a3.in-" (at 196.85 105.41 180) (fields_autoplaced)
     (effects (font (size 1.27 1.27)) (justify right bottom))
   )
@@
     (effects (font (size 1.27 1.27)) (justify right bottom))
   )
-  (label "usb1.d-" (at 44.45 90.17 0)
+  (label "usb1.d-" (at 44.45 90.17 0) (fields_autoplaced)
     (effects (font (size 1.27 1.27)) (justify left bottom))
   )
