File: projects/word_watch/word_watch.kicad_sch (KiCad schematic)
At the start: 0 parts

Commit message: finish word_watch
Parts:
- added BT1: CR2032, Battery:BatteryHolder_Keystone_1060_1x2032, symbol Device:Battery_Cell
- added C1, C5: 4u7, Capacitor_SMD:C_0402_1005Metric, symbol Device:C_Small
- added C2, C6: 100n, Capacitor_SMD:C_0402_1005Metric, symbol Device:C_Small
- added C3, C4: 20p, Capacitor_SMD:C_0402_1005Metric, symbol Device:C_Small
- added D1: charge, LED_SMD:LED_0402_1005Metric, symbol Device:LED_Small_Filled
- added D10, D11, D12, D13, D14, D15, D16, D17, D18, D19, D20, D21, D22, D23, D24, D25, D26, D27, D28, D29, D3, D30, D31, D32, D33, D34, D35, D36, D37, D38, D39, D4, D40, D41, D42, D43, D44, D45, D46, D47, D48, D49, D5, D50, D51, D52, D53, D54, D55, D56, D57, D58, D59, D6, D60, D61, D62, D63, D64, D65, D66, D67, D68, D69, D7, D70, D71, D72, D73, D74, D75, D76, D77, D78, D79, D8, D80, D81, D82, D83, D84, D85, D86, D87, D88, D89, D9, D90, D91, D92: LED_Small_Filled, LED_SMD:LED_0402_1005Metric, symbol Device:LED_Small_Filled
- added D2: full, LED_SMD:LED_0402_1005Metric, symbol Device:LED_Small_Filled
- added J1: charge, extraparts:USB_Micro-B_U254-05, symbol Connector:USB_B_Micro
- added J2: updi/uart, Connector:Tag-Connect_TC2030-IDC-NL_2x03_P1.27mm_Vertical, symbol Connector_Generic:Conn_02x03_Odd_Even
- added R1: 10k, Resistor_SMD:R_0402_1005Metric, symbol Device:R_Small
- added R10, R11, R12, R13, R4, R5, R6, R7, R8, R9: 22, Resistor_SMD:R_0402_1005Metric, symbol Device:R_Small
- added R2, R3: 2k2, Resistor_SMD:R_0402_1005Metric, symbol Device:R_Small
- added SW1: btn_up, Button_Switch_SMD:SW_SPST_PTS810, symbol Switch:SW_SPST
- added SW2: btn_down, Button_Switch_SMD:SW_SPST_PTS810, symbol Switch:SW_SPST
- added SW3: btn_wake, Button_Switch_SMD:SW_SPST_PTS810, symbol Switch:SW_SPST
- added SW4: SW-18020P, Crystal:Crystal_AT310_D3.0mm_L10.0mm_Horizontal, symbol Switch:SW_Reed
- added U1: MCP73831-2-OT, Package_TO_SOT_SMD:SOT-23-5, symbol Battery_Management:MCP73831-2-OT
- added U2: TG-3541CE, extraparts:Crystal_SMD_SeikoEpson_TG-3541CE-10Pin_3.2x2.5mm, symbol extraparts:TG-3541CE
- added U3: ATtiny1616-M, Package_DFN_QFN:VQFN-20-1EP_3x3mm_P0.4mm_EP1.7x1.7mm, symbol MCU_Microchip_ATtiny:ATtiny1616-M
- added Y1: 32.768kHz, Crystal:Crystal_SMD_MicroCrystal_CM9V-T1A-2Pin_1.6x1.0mm, symbol Device:Crystal_Small
Connections:
- new net: D1.1 (K), R2.2
- new net: R2.1, R3.1, U1.1 (STAT)
- new net: D2.2 (A), R3.2
- new net: R1.1, U1.5 (PROG)
- new net +5V: C1.1, D1.2 (A), J1.1 (VBUS), U1.4 (V_{DD})
- new net +BATT: BT1.1 (+), C2.1, C5.1, C6.1, J2.1 (Pin_1), U1.3 (V_{BAT}), U2.1 (OE), U2.2 (Vcc), U2.3 (Vcc), U3.4 (VCC)
- new net GND: BT1.2 (-), C1.2, C2.2, C3.1, C4.2, C5.2, C6.2, D2.1 (K), J1.5 (GND), J1.6 (Shield), J2.3 (Pin_3), R1.2, SW1.1 (A), SW2.1 (A), SW3.1 (A), SW4.2, U1.2 (V_{SS}), U2.5 (GND), U2.7 (GND), U2.8 (GND), U2.9 (GND), U3.21 (GND), U3.3 (GND)
- new net btn_down: SW3.2 (B), U3.18 (PC3)
- new net btn_up: SW1.2 (B), U3.16 (PC1)
- new net btn_wake: SW2.2 (B), U3.17 (PC2)
- new net led1: R4.1, U3.6 (PA5)
- new net led10: R13.1, U3.14 (PB0)
- new net led2: R5.1, U3.7 (PA6)
- new net led3: R6.1, U3.8 (PA7)
- new net led4: R7.1, U3.9 (PB5)
- new net led5: R8.1, U3.10 (PB4)
- new net led6: R9.1, U3.5 (PA4)
- new net led7: R10.1, U3.2 (PA3)
- new net led8: R11.1, U3.1 (PA2)
- new net led9: R12.1, U3.13 (PB1)
- new net rled1: D12.1 (K), D21.1 (K), D22.1 (K), D23.1 (K), D24.1 (K), D25.1 (K), D26.1 (K), D27.1 (K), D28.1 (K), D29.2 (A), D3.2 (A), D30.2 (A), D31.2 (A), D32.2 (A), D33.2 (A), D34.2 (A), D35.2 (A), D36.2 (A), R4.2
- new net rled10: D10.1 (K), D11.1 (K), D12.2 (A), D13.2 (A), D14.2 (A), D15.2 (A), D16.2 (A), D17.2 (A), D18.2 (A), D19.2 (A), D20.2 (A), D3.1 (K), D4.1 (K), D5.1 (K), D6.1 (K), D7.1 (K), D8.1 (K), D9.1 (K), R13.2
- new net rled2: D13.1 (K), D21.2 (A), D29.1 (K), D37.1 (K), D38.1 (K), D39.1 (K), D4.2 (A), D40.1 (K), D41.1 (K), D42.1 (K), D43.1 (K), D44.2 (A), D45.2 (A), D46.2 (A), D47.2 (A), D48.2 (A), D49.2 (A), D50.2 (A), R5.2
- new net rled3: D14.1 (K), D22.2 (A), D30.1 (K), D37.2 (A), D44.1 (K), D5.2 (A), D51.1 (K), D52.1 (K), D53.1 (K), D54.1 (K), D55.1 (K), D56.1 (K), D57.2 (A), D58.2 (A), D59.2 (A), D60.2 (A), D61.2 (A), D62.2 (A), R6.2
- new net rled4: D15.1 (K), D23.2 (A), D31.1 (K), D38.2 (A), D45.1 (K), D51.2 (A), D57.1 (K), D6.2 (A), D63.1 (K), D64.1 (K), D65.1 (K), D66.1 (K), D67.1 (K), D68.2 (A), D69.2 (A), D70.2 (A), D71.2 (A), D72.2 (A), R7.2
- new net rled5: D16.1 (K), D24.2 (A), D32.1 (K), D39.2 (A), D46.1 (K), D52.2 (A), D58.1 (K), D63.2 (A), D68.1 (K), D7.2 (A), D73.1 (K), D74.1 (K), D75.1 (K), D76.1 (K), D77.2 (A), D78.2 (A), D79.2 (A), D80.2 (A), R8.2
- new net rled6: D17.1 (K), D25.2 (A), D33.1 (K), D40.2 (A), D47.1 (K), D53.2 (A), D59.1 (K), D64.2 (A), D69.1 (K), D73.2 (A), D77.1 (K), D8.2 (A), D81.1 (K), D82.1 (K), D83.1 (K), D84.2 (A), D85.2 (A), D86.2 (A), R9.2
- new net rled7: D18.1 (K), D26.2 (A), D34.1 (K), D41.2 (A), D48.1 (K), D54.2 (A), D60.1 (K), D65.2 (A), D70.1 (K), D74.2 (A), D78.1 (K), D81.2 (A), D84.1 (K), D87.1 (K), D88.1 (K), D89.2 (A), D9.2 (A), D90.2 (A), R10.2
- new net rled8: D10.2 (A), D19.1 (K), D27.2 (A), D35.1 (K), D42.2 (A), D49.1 (K), D55.2 (A), D61.1 (K), D66.2 (A), D71.1 (K), D75.2 (A), D79.1 (K), D82.2 (A), D85.1 (K), D87.2 (A), D89.1 (K), D91.1 (K), D92.2 (A), R11.2
- new net rled9: D11.2 (A), D20.1 (K), D28.2 (A), D36.1 (K), D43.2 (A), D50.1 (K), D56.2 (A), D62.1 (K), D67.2 (A), D72.1 (K), D76.2 (A), D80.1 (K), D83.2 (A), D86.1 (K), D88.2 (A), D90.1 (K), D91.2 (A), D92.1 (K), R12.2
- new net shake_wake: SW4.1, U3.15 (PC0)
- new net tx: J2.2 (Pin_2), U3.20 (PA1)
- new net updi: J2.6 (Pin_6), U3.19 (~{RESET}/PA0)
- new net xtal_in: C3.2, U2.4 (OUT), U3.11 (PB3), Y1.2
- new net xtal_out: C4.1, U3.12 (PB2), Y1.1
- no-connect marks 0 -> 5
Other:
- note added: "charlieplex matrix"
- note added: "clock"
- note added: "crystal ($) - 20ppm => ~10min/year tcxo ($$$) - 2ppm => ~1min/year"
- note added: "debug/ui"
- note added: "measure vbat w/ internal vref"
- note added: "micro"
- note added: "power"
- note added: "~100mA"
