File: breakouts/adin1110_oaspi/adin1110_oaspi.kicad_sch (KiCad schematic)
At the start: 66 parts, among them J1 USB_B_Micro, J2 swd/uart, J3 Conn_01x02_MountingPin, SW1 boot, U1 MIC5365-3.3YC5, U2 LPC1549JBD48, U3 ADIN1110, Y1 12MHz, Y2 25MHz

Commit message: minor updates
Parts:
- R18, R19, R3, R4, R5: value 220 -> 4k7
Changed lines of the file:
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@@
 			)
 		)
-		(property "Value" "220"
+		(property "Value" "4k7"
 			(at 94.615 149.225 90)
 			(effects
@@
 			)
 		)
-		(property "Value" "220"
+		(property "Value" "4k7"
 			(at 94.615 159.385 90)
 			(effects
@@
 			)
 		)
-		(property "Value" "220"
+		(property "Value" "4k7"
 			(at 249.555 101.6 90)
 			(effects
@@
 			)
 		)
-		(property "Value" "220"
+		(property "Value" "4k7"
 			(at 249.555 97.79 90)
 			(effects
@@
 			)
 		)
-		(property "Value" "220"
+		(property "Value" "4k7"
 			(at 94.615 154.305 90)
 			(effects
