File: breakouts/ncn26010_oaspi/ncn26010_oaspi.kicad_sch (KiCad schematic)
At the start: 59 parts, among them J1 USB_B_Micro, J2 swd/uart, J3 Conn_01x04_MountingPin, SW1 boot, U1 MIC5365-3.3YC5, U2 LPC1549JBD48, U3 NCN26010, Y1 12MHz, Y2 25MHz

Commit message: minor updates
Parts:
- R18, R19: value 2k2 -> 10k
- R3, R4, R5: value 220 -> 10k
Changed lines of the file:
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@@
 			)
 		)
-		(property "Value" "220"
+		(property "Value" "10k"
 			(at 104.775 155.575 90)
 			(effects
@@
 			)
 		)
-		(property "Value" "220"
+		(property "Value" "10k"
 			(at 104.775 165.735 90)
 			(effects
@@
 			)
 		)
-		(property "Value" "2k2"
+		(property "Value" "10k"
 			(at 244.475 105.41 90)
 			(effects
@@
 			)
 		)
-		(property "Value" "220"
+		(property "Value" "10k"
 			(at 104.775 160.655 90)
 			(effects
@@
 			)
 		)
-		(property "Value" "2k2"
+		(property "Value" "10k"
 			(at 244.475 101.6 90)
 			(effects
